File: cpOD.sch (EAGLE design)
At the start: 29 parts, among them IC1 LM358D, Q1 2N7002

Commit message: 2.0B-WIP
Parts:
- added R11: 10K, SPCoast:R-POTENTIOMETERPT-10S
- added R12: 10K, SPCoast:R-POTENTIOMETERTC33X
- C2: value 1uF -> 1.0uF
- R1: value 2.2M -> 2M2
- R10: value 10k -> 3K3
- R2, R3, R6: value 10k -> 10K
- R7: value 3.3k -> 1M
- R8: value 1M -> 10K; device SPCoast:R0603-RES -> SPCoast:R-POTENTIOMETERETB
- R9: value 10k -> 10K; device SPCoast:R-POTENTIOMETERTC33X -> SPCoast:R0603-RES
Connections:
- net DETECTED: now also R10.2, R7.1; no longer R7.2, R8.1
- net GND: now also R11.E, R12.E, R8.E; no longer R9.E
- net N$11: now also R10.1; no longer R7.1
- net SENS+: now also R11.A, R12.A, R8.A, R9.1; no longer R10.1, R9.A
- net SENSITIVITY: now also R11.S, R12.S, R7.2, R8.S; no longer R8.2, R9.S
- net V+: now also R9.2; no longer R10.2
Other:
- moved on the sheet: R10, R7
Changed lines of the file:
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@@
 <layer number="18" name="Vias" color="1" fill="1" visible="yes" active="no"/>
 <layer number="19" name="Unrouted" color="6" fill="1" visible="yes" active="no"/>
-<layer number="20" name="Dimension" color="36" fill="1" visible="yes" active="no"/>
-<layer number="21" name="tPlace" color="36" fill="1" visible="yes" active="no"/>
-<layer number="22" name="bPlace" color="17" fill="1" visible="yes" active="no"/>
+<layer number="20" name="Dimension" color="15" fill="1" visible="yes" active="no"/>
+<layer number="21" name="tPlace" color="22" fill="1" visible="yes" active="no"/>
+<layer number="22" name="bPlace" color="22" fill="1" visible="yes" active="no"/>
 <layer number="23" name="tOrigins" color="30" fill="1" visible="yes" active="no"/>
 <layer number="24" name="bOrigins" color="15" fill="1" visible="yes" active="no"/>
 <layer number="25" name="tNames" color="36" fill="1" visible="yes" active="no"/>
 <layer number="26" name="bNames" color="34" fill="1" visible="yes" active="no"/>
-<layer number="27" name="tValues" color="23" fill="1" visible="yes" active="no"/>
+<layer number="27" name="tValues" color="22" fill="1" visible="yes" active="no"/>
 <layer number="28" name="bValues" color="7" fill="1" visible="yes" active="no"/>
 <layer number="29" name="tStop" color="5" fill="1" visible="no" active="no"/>
@@
 <layer number="46" name="Milling" color="11" fill="1" visible="yes" active="no"/>
 <layer number="47" name="Measures" color="21" fill="1" visible="yes" active="no"/>
-<layer number="48" name="Document" color="47" fill="1" visible="yes" active="no"/>
+<layer number="48" name="Document" color="49" fill="1" visible="yes" active="no"/>
 <layer number="49" name="Reference" color="7" fill="1" visible="yes" active="no"/>
 <layer number="50" name="dxf" color="7" fill="1" visible="yes" active="no"/>
@@
 <part name="C1" library="SPCoast" deviceset="CAP*" device="0603" value="0.1uF"/>
 <part name="C4" library="SPCoast" deviceset="CAP*" device="0603" value="0.1uF"/>
-<part name="C2" library="SPCoast" deviceset="CAP*" device="0603" value="1uF"/>
+<part name="C2" library="SPCoast" deviceset="CAP*" device="0603" value="1.0uF"/>
 <part name="C3" library="SPCoast" deviceset="CAP*" device="0603" value="0.01uF"/>
-<part name="R3" library="SPCoast" deviceset="R*" device="0603-RES" value="10k"/>
-<part name="R6" library="SPCoast" deviceset="R*" device="0603-RES" value="10k"/>
+<part name="R3" library="SPCoast" deviceset="R*" device="0603-RES" value="10K"/>
+<part name="R6" library="SPCoast" deviceset="R*" device="0603-RES" value="10K"/>
 <part name="IC1" library="SPCoast" deviceset="LM6132A" device="" value="LM358D"/>
 <part name="R4" library="SPCoast" deviceset="R*" device="0603-RES" value="200R"/>
@@
 <part name="P+1" library="supply1" deviceset="V+" device=""/>
 <part name="GND3" library="supply1" deviceset="GND" device=""/>
-<part name="R10" library="SPCoast" deviceset="R*" device="0603-RES" value="10k"/>
-<part name="R8" library="SPCoast" deviceset="R*" device="0603-RES" value="1M"/>
+<part name="R9" library="SPCoast" deviceset="R*" device="0603-RES" value="10K"/>
+<part name="R7" library="SPCoast" deviceset="R*" device="0603-RES" value="1M"/>
 <part name="GND4" library="supply1" deviceset="GND" device=""/>
-<part name="R2" library="SPCoast" deviceset="R*" device="0603-RES" value="10k"/>
-<part name="R1" library="SPCoast" deviceset="R*" device="0603-RES" value="2.2M"/>
+<part name="R2" library="SPCoast" deviceset="R*" device="0603-RES" value="10K"/>
+<part name="R1" library="SPCoast" deviceset="R*" device="0603-RES" value="2M2"/>
 <part name="GND5" library="supply1" deviceset="GND" device=""/>
 <part name="GND6" library="supply1" deviceset="GND" device=""/>
 <part name="Q1" library="SPCoast" deviceset="MOSFET-N-*-?" device="SOT23" technology="2N7002" value="2N7002"/>
 <part name="GND7" library="supply1" deviceset="GND" device=""/>
-<part name="R7" library="SPCoast" deviceset="R*" device="0603-RES" value="3.3k"/>
+<part name="R10" library="SPCoast" deviceset="R*" device="0603-RES" value="3K3"/>
 <part name="LED1" library="SPCoast" deviceset="LED*" device="0603-LED" value="Y"/>
 <part name="GND12" library="supply1" deviceset="GND" device=""/>
@@
 <part name="GND9" library="supply1" deviceset="GND" device=""/>
 <part name="J1" library="SPCoast" deviceset="CONNECTOR-M05" device="1.56"/>
-<part name="R9" library="SPCoast" deviceset="R-POTENTIOMETER" device="TC33X" value="10k"/>
+<part name="R8" library="SPCoast" deviceset="R-POTENTIOMETER" device="ETB" value="10K"/>
 <part name="U$5" library="SPCoast" deviceset="MOUNTINGHOLE" device="L"/>
 <part name="U$6" library="SPCoast" deviceset="MOUNTINGHOLE" device="L"/>
@@
 <part name="GND11" library="supply1" deviceset="GND" device=""/>
 <part name="J2" library="SPCoast" deviceset="CONNECTOR-M05" device="PTH"/>
+<part name="R11" library="SPCoast" deviceset="R-POTENTIOMETER" device="PT-10S" value="10K"/>
+<part name="R12" library="SPCoast" deviceset="R-POTENTIOMETER" device="TC33X" value="10K"/>
 </parts>
 <sheets>
@@
 <attribute name="VALUE" x="96.52" y="12.7" size="1.778" layer="96"/>
 </instance>
-<instance part="R10" gate="R" x="127" y="124.46" smashed="yes" rot="R90">
+<instance part="R9" gate="R" x="127" y="124.46" smashed="yes" rot="R90">
 <attribute name="NAME" x="124.46" y="126.7714" size="1.778" layer="95" rot="R180"/>
 <attribute name="VALUE" x="125.73" y="123.952" size="1.778" layer="96" rot="R180"/>
 </instance>
-<instance part="R8" gate="R" x="148.59" y="111.76" smashed="yes" rot="R180">
+<instance part="R7" gate="R" x="148.59" y="111.76" smashed="yes" rot="R180">
 <attribute name="NAME" x="149.86" y="115.3414" size="1.778" layer="95" rot="R180"/>
 <attribute name="VALUE" x="149.86" y="109.982" size="1.778" layer="96" rot="R180"/>
@@
 <attribute name="VALUE" x="154.94" y="81.28" size="1.778" layer="96"/>
 </instance>
-<instance part="R7" gate="R" x="185.42" y="88.9" smashed="yes" rot="R90">
+<instance part="R10" gate="R" x="185.42" y="88.9" smashed="yes" rot="R90">
 <attribute name="NAME" x="193.04" y="89.9414" size="1.778" layer="95" rot="R180"/>
 <attribute name="VALUE" x="194.31" y="87.122" size="1.778" layer="96" rot="R180"/>
@@
 </instance>
 <instance part="J1" gate="CON1" x="17.78" y="142.24"/>
-<instance part="R9" gate="1" x="127" y="111.76" rot="MR270"/>
+<instance part="R8" gate="1" x="127" y="111.76" rot="MR270"/>
 <instance part="U$5" gate="MT1" x="241.3" y="35.56"/>
 <instance part="U$6" gate="MT1" x="231.14" y="35.56"/>
@@
 </instance>
 <instance part="J2" gate="CON1" x="12.7" y="33.02"/>
+<instance part="R11" gate="1" x="127" y="111.76" rot="MR270"/>
+<instance part="R12" gate="1" x="127" y="111.76" rot="MR270"/>
 </instances>
 <busses>
@@
 <segment>
 <pinref part="GND4" gate="1" pin="GND"/>
-<pinref part="R9" gate="1" pin="E"/>
+<pinref part="R8" gate="1" pin="E"/>
 <wire x1="127" y1="106.68" x2="127" y2="58.42" width="0.1524" layer="91"/>
+<pinref part="R11" gate="1" pin="E"/>
+<junction x="127" y="106.68"/>
+<pinref part="R12" gate="1" pin="E"/>
 </segment>
 <segment>
@@
 <segment>
 <pinref part="P+6" gate="1" pin="V+"/>
-<pinref part="R10" gate="R" pin="2"/>
+<pinref part="R9" gate="R" pin="2"/>
 <wire x1="127" y1="129.54" x2="127" y2="137.16" width="0.1524" layer="91"/>
 </segment>
@@
 <segment>
 <wire x1="127" y1="116.84" x2="127" y2="119.38" width="0.1524" layer="91"/>
-<pinref part="R10" gate="R" pin="1"/>
+<pinref part="R9" gate="R" pin="1"/>
 <label x="124.46" y="105.41" size="1.016" layer="95" rot="R270"/>
-<pinref part="R9" gate="1" pin="A"/>
+<pinref part="R8" gate="1" pin="A"/>
+<pinref part="R11" gate="1" pin="A"/>
+<junction x="127" y="116.84"/>
+<pinref part="R12" gate="1" pin="A"/>
 </segment>
 </net>
@@
 <wire x1="143.51" y1="111.76" x2="142.24" y2="111.76" width="0.1524" layer="91"/>
 <pinref part="IC1" gate="B" pin="+IN"/>
-<pinref part="R8" gate="R" pin="2"/>
+<pinref part="R7" gate="R" pin="2"/>
 <label x="133.35" y="113.03" size="1.016" layer="95"/>
-<pinref part="R9" gate="1" pin="S"/>
+<pinref part="R8" gate="1" pin="S"/>
 <wire x1="142.24" y1="111.76" x2="142.24" y2="101.6" width="0.1524" layer="91"/>
 <wire x1="132.08" y1="111.76" x2="142.24" y2="111.76" width="0.1524" layer="91"/>
 <junction x="142.24" y="111.76"/>
+<pinref part="R11" gate="1" pin="S"/>
+<junction x="132.08" y="111.76"/>
+<pinref part="R12" gate="1" pin="S"/>
 </segment>
 </net>
@@
 <pinref part="R1" gate="R" pin="2"/>
 <pinref part="IC1" gate="B" pin="OUT"/>
-<pinref part="R8" gate="R" pin="1"/>
-<pinref part="R7" gate="R" pin="2"/>
+<pinref part="R7" gate="R" pin="1"/>
+<pinref part="R10" gate="R" pin="2"/>
 <pinref part="D1" gate="G$1" pin="COM"/>
 <wire x1="185.42" y1="99.06" x2="185.42" y2="109.22" width="0.1524" layer="91"/>
@@
 <segment>
 <wire x1="185.42" y1="83.82" x2="185.42" y2="71.12" width="0.1524" layer="91"/>
-<pinref part="R7" gate="R" pin="1"/>
+<pinref part="R10" gate="R" pin="1"/>
 <pinref part="LED1" gate="LED" pin="A"/>
 </segment>

Commit message: Version 1.1
Parts:
- C1: value 0.1uF -> 1.0uF
- C2: value 1.0uF -> 0.01uF
- C3: value 0.01uF -> 0.1uF
- D2: value BAT54A -> BAT54C; device SPCoast:DIODE-BAT54A23 -> SPCoast:DIODE-BAT54C23
- D3: value BAT54C -> BAT54A; device SPCoast:DIODE-BAT54C23 -> SPCoast:DIODE-BAT54A23
- J1: device SPCoast:CONNECTOR-M051.56 -> SPCoast:CONNECTOR-M05PTH
- J2: device SPCoast:CONNECTOR-M05PTH -> SPCoast:CONNECTOR-M051.56
- R10: value 3K3 -> 2k2
- R7: value 1M -> 10K
- R8: value 10K -> 1M; device SPCoast:R-POTENTIOMETERETB -> SPCoast:R0603-RES
- R9: device SPCoast:R0603-RES -> SPCoast:R-POTENTIOMETERETB
- renumbered U$5 to U$1, U$6 to U$2
Connections:
- net !VOUT: now also J1.3, J2.5; no longer J1.5, J2.3
- net DCC-A: now also J2.2; no longer J1.2
- net DCC-B: now also J2.4; no longer J1.4
- net DETECTED: now also R8.1; no longer R7.1
- net GND: now also C3.2, R9.E; no longer C2.2, R8.E
- net INPUT-A: now also D2.A1, D3.C2, J1.4; no longer D2.C2, D3.A1, J2.4
- net INPUT-B: now also D2.A2, D3.C1, J1.5; no longer D2.C1, D3.A2, J2.5
- net OCCUPIED: now also C1.1; no longer C2.1
- net SENS+: now also R7.1, R9.A; no longer R8.A, R9.1
- net SENSITIVITY: now also R8.2, R9.S; no longer R7.2, R8.S
- net STAGE1+: now also C3.1; no longer C4.1
- net STAGE1-: now also C2.1; no longer C3.1
- net TRIGGERED: now also C2.2; no longer C3.2
- net V+: now also C4.1, J1.2, J2.3, R7.2; no longer C1.1, J1.3, J2.2, R9.2
Other:
- moved on the sheet: C1, C2, C3, C4, D4, IC1A, IC1B, J1, J2, R11, R12, R3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

Commit message: Version 2.0
Parts:
- removed FID1, FID2: FIDUCIAL, SPCoast:FIDUCIAL
- removed U$2: MOUNTINGHOLEL, SPCoast:MOUNTINGHOLEL
- added MH2: MOUNTINGHOLEL, SPCoast:MOUNTINGHOLEL
- renumbered U$1 to MH1
Other:
- note added: "C"
- note removed: "A"
Changed lines of the file:
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@@
 <part name="J2" library="SPCoast" deviceset="CONNECTOR-M05" device="1.56"/>
 <part name="R9" library="SPCoast" deviceset="R-POTENTIOMETER" device="ETB" value="10K"/>
-<part name="U$1" library="SPCoast" deviceset="MOUNTINGHOLE" device="L"/>
-<part name="U$2" library="SPCoast" deviceset="MOUNTINGHOLE" device="L"/>
+<part name="MH1" library="SPCoast" deviceset="MOUNTINGHOLE" device="L"/>
+<part name="MH2" library="SPCoast" deviceset="MOUNTINGHOLE" device="L"/>
 <part name="P+5" library="supply1" deviceset="V+" device=""/>
 <part name="P+6" library="supply1" deviceset="V+" device=""/>
 <part name="P+7" library="supply1" deviceset="V+" device=""/>
-<part name="FID1" library="SPCoast" deviceset="FIDUCIAL" device=""/>
-<part name="FID2" library="SPCoast" deviceset="FIDUCIAL" device=""/>
 <part name="X2" library="SPCoast" deviceset="PULSE-TRANSFORMER" device="M"/>
 <part name="P+8" library="supply1" deviceset="V+" device=""/>
@@
 14v p/p @ 5A</text>
 <text x="238.76" y="12.7" size="2.54" layer="91">2.0</text>
-<text x="240.03" y="6.35" size="2.54" layer="91">A</text>
+<text x="240.03" y="6.35" size="2.54" layer="91">C</text>
 <text x="165.1" y="6.35" size="2.54" layer="91">John Plocher, 2021.08</text>
 <text x="214.376" y="10.922" size="1.778" layer="91">cpOD &amp; DCCOD</text>
@@
 <instance part="J2" gate="CON1" x="17.78" y="142.24"/>
 <instance part="R9" gate="1" x="133.35" y="111.76" rot="MR270"/>
-<instance part="U$1" gate="MT1" x="241.3" y="35.56"/>
-<instance part="U$2" gate="MT1" x="231.14" y="35.56"/>
+<instance part="MH1" gate="MT1" x="241.3" y="35.56"/>
+<instance part="MH2" gate="MT1" x="241.3" y="43.18"/>
 <instance part="P+5" gate="1" x="99.06" y="35.56" smashed="yes">
 <attribute name="VALUE" x="100.33" y="38.1" size="1.778" layer="96" rot="R180"/>
@@
 <attribute name="VALUE" x="165.1" y="142.24" size="1.778" layer="96" rot="R180"/>
 </instance>
-<instance part="FID1" gate="FID1" x="241.3" y="45.72"/>
-<instance part="FID2" gate="FID1" x="228.6" y="45.72"/>
 <instance part="X2" gate="X1" x="33.02" y="78.74" rot="MR180"/>
 <instance part="P+8" gate="1" x="33.02" y="33.02" smashed="yes">
